File: OpenTimeWatch-1.kicad_sch (KiCad schematic)
At the start: 38 parts, among them J1 1.44" LCD, J2 USB_B_Micro, J3 Speaker, J4 MPU6050, J5 Battery, Q1 Si2319CDS, SW1 Right, SW2 Left down, SW3 Left up, SW4 SW_DIP_x01, U1 ESP32-S3-WROOM-1, U2 TP4056-42-ESOP8, U3 RT9701

Commit message: Update PCB schematics and design files
Parts:
- added J6: UART, Connector_PinSocket_2.54mm:PinSocket_1x02_P2.54mm_Vertical, symbol Connector:Conn_01x02_Socket
- added J7: Heart Rate Sensor, symbol Connector:Conn_01x01_Socket
- added R11: 100k, symbol Device:R_US
Connections:
- net at U2.7 (~{CHRG}): now also R11.1
- net GPIO17: now reaches U1.10 (IO17)
- net GPIO17: now also J6.1 (Pin_1), J7.1 (Pin_1)
- net GPIO18: now reaches U1.11 (IO18)
- net GPIO46: now reaches U1.16 (IO46)
- net GPIO46: now also R11.2
- net GPIO7: now reaches U1.7 (IO7)
- net GPIO7: now also J6.2 (Pin_2)
Other:
- moved on the sheet: J3, R2

Commit message: Add files via upload
Connections:
- net GND: now also U2.9 (EPAD)
Other:
- moved on the sheet: R11
Changed lines of the file:
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@@
 	(wire
 		(pts
+			(xy 52.07 120.65) (xy 52.07 135.89)
+		)
+		(stroke
+			(width 0)
+			(type default)
+		)
+	)
+	(wire
+		(pts
 			(xy 152.4 123.19) (xy 176.53 123.19)
 		)
@@
 	(wire
 		(pts
-			(xy 49.53 120.65) (xy 49.53 135.89)
-		)
-		(stroke
-			(width 0)
-			(type default)
-		)
-	)
-	(wire
-		(pts
 			(xy 110.49 99.06) (xy 118.11 99.06)
 		)
@@
 	(wire
 		(pts
+			(xy 60.96 120.65) (xy 63.5 120.65)
+		)
+		(stroke
+			(width 0)
+			(type default)
+		)
+	)
+	(wire
+		(pts
 			(xy 167.64 120.65) (xy 176.53 120.65)
 		)
@@
 	(wire
 		(pts
-			(xy 53.34 104.14) (xy 49.53 104.14)
+			(xy 53.34 104.14) (xy 52.07 104.14)
 		)
 		(stroke
@@
 	(wire
 		(pts
-			(xy 49.53 104.14) (xy 49.53 113.03)
+			(xy 52.07 104.14) (xy 52.07 113.03)
 		)
 		(stroke
@@
 	(wire
 		(pts
+			(xy 60.96 116.84) (xy 60.96 120.65)
+		)
+		(stroke
+			(width 0)
+			(type default)
+		)
+	)
+	(wire
+		(pts
 			(xy 167.64 57.15) (xy 173.99 57.15)
 		)
@@
 	(global_label "GPIO46"
 		(shape input)
-		(at 49.53 135.89 270)
+		(at 52.07 135.89 270)
 		(fields_autoplaced yes)
 		(effects
@@
 		)
 		(property "Intersheetrefs" "${INTERSHEET_REFS}"
-			(at 49.53 145.7695 90)
+			(at 52.07 145.7695 90)
 			(effects
 				(font
@@
 	(symbol
 		(lib_id "Device:R_US")
-		(at 49.53 116.84 0)
+		(at 52.07 116.84 0)
 		(unit 1)
 		(exclude_from_sim no)
@@
 		(dnp no)
 		(property "Reference" "R11"
-			(at 52.07 115.5699 0)
+			(at 54.61 115.5699 0)
 			(effects
 				(font
@@
 		)
 		(property "Value" "100k"
-			(at 51.308 117.602 0)
+			(at 53.848 117.602 0)
 			(effects
 				(font
@@
 		)
 		(property "Footprint" ""
-			(at 50.546 117.094 90)
+			(at 53.086 117.094 90)
 			(effects
 				(font
@@
 		)
 		(property "Datasheet" "~"
-			(at 49.53 116.84 0)
+			(at 52.07 116.84 0)
 			(effects
 				(font
@@
 		)
 		(property "Description" "Resistor, US symbol"
-			(at 49.53 116.84 0)
+			(at 52.07 116.84 0)
 			(effects
 				(font
